Commit message: Update model.xacro

File: manipualtor/urdf/model.xacro (robot description, xacro)
@@ -110,4 +110,26 @@
     <limit effort="0.245166" lower="-1.57" upper="1.57" velocity="0.5"/>
   </joint>
+  <!-- imu_block1 -->
+  <link name="imu_block1">
+    <collision>
+      <origin xyz="0 0 0" rpy="0 0 0"/>
+      <geometry>
+        <box size="0.015 0.025 0.005"/>
+      </geometry>
+    </collision>
+    <visual>
+      <origin xyz="0 0 0" rpy="0 0 0"/>
+      <geometry>
+        <box size="0.015 0.025 0.005"/>
+      </geometry>
+      <material name="black"/>
+    </visual>
+    <xacro:default_inertial mass="1e-5"/>
+  </link>
+  <joint name="link1_to_imu_block1" type="fixed">
+    <origin xyz="${link1_r/2 + 0.015 + 0.015/2} 0 ${link1_l/2 + 0.005/2}" rpy="0 0 0"/>
+    <parent link="link1"/>
+    <child link="imu_block1"/>
+  </joint>
   <!-- for_link2_1 -->
   <link name="for_link2_1">
@@ -178,25 +200,47 @@
     <axis xyz="0 1 0"/>
   </joint>
-  <!-- imu_block -->
-  <link name="imu_block">
-    <collision>
-      <origin xyz="0 0 0" rpy="0 0 0"/>
-      <geometry>
-        <box size="0.001 0.005 0.002"/>
-      </geometry>
-    </collision>
-    <visual>
-      <origin xyz="0 0 0" rpy="0 0 0"/>
-      <geometry>
-        <box size="0.001 0.005 0.002"/>
-      </geometry>
-      <material name="black"/>
-    </visual>
-    <xacro:default_inertial mass="1e-5"/>
-  </link>
-  <joint name="link2_to_imu_block" type="fixed">
-    <origin xyz="${0.017 + 0.0125} ${-link2_d + link1_r} 0.046" rpy="0 0 0"/>
+  <!-- imu_block2 -->
+  <link name="imu_block2">
+    <collision>
+      <origin xyz="0 0 0" rpy="0 0 0"/>
+      <geometry>
+        <box size="0.015 0.025 0.005"/>
+      </geometry>
+    </collision>
+    <visual>
+      <origin xyz="0 0 0" rpy="0 0 0"/>
+      <geometry>
+        <box size="0.015 0.025 0.005"/>
+      </geometry>
+      <material name="black"/>
+    </visual>
+    <xacro:default_inertial mass="1e-5"/>
+  </link>
+  <joint name="link2_to_imu_block2" type="fixed">
+    <origin xyz="0 ${0.025/2 + link2_d/2} 0" rpy="0 ${3.14/2 + 3.14/6} 0"/>
     <parent link="link2"/>
-    <child link="imu_block"/>
+    <child link="imu_block2"/>
+  </joint>
+  <!-- laser1 -->
+  <link name="laser1">
+    <collision>
+      <origin xyz="0 0 0" rpy="0 0 0"/>
+      <geometry>
+        <box size="0.001 0.005 0.002"/>
+      </geometry>
+    </collision>
+    <visual>
+      <origin xyz="0 0 0" rpy="0 0 0"/>
+      <geometry>
+        <box size="0.001 0.005 0.002"/>
+      </geometry>
+      <material name="black"/>
+    </visual>
+    <xacro:default_inertial mass="1e-5"/>
+  </link>
+  <joint name="link2_to_laser1" type="fixed">
+    <origin xyz="${0.017 + 0.0125} ${-link2_d + link1_r} 0.046" rpy="0 ${3.14 + 3.14/2/2/2} 0"/>
+    <parent link="link2"/>
+    <child link="laser1"/>
   </joint>
   <!-- link3 -->
@@ -226,4 +270,26 @@
     <axis xyz="0 1 0"/>
   </joint>
+  <!-- imu_block3 -->
+  <link name="imu_block3">
+    <collision>
+      <origin xyz="0 0 0" rpy="0 0 0"/>
+      <geometry>
+        <box size="0.025 0.015 0.005"/>
+      </geometry>
+    </collision>
+    <visual>
+      <origin xyz="0 0 0" rpy="0 0 0"/>
+      <geometry>
+        <box size="0.025 0.015 0.005"/>
+      </geometry>
+      <material name="black"/>
+    </visual>
+    <xacro:default_inertial mass="1e-5"/>
+  </link>
+  <joint name="link3_to_imu_block3" type="fixed">
+    <origin xyz="${-0.025/2} ${link3_d/2} ${link3_h - 0.005}" rpy="0 0 0"/>
+    <parent link="link3"/>
+    <child link="imu_block3"/>
+  </joint>
  <!-- link4 -->
   <link name="link4">
@@ -273,4 +339,26 @@
     <child link="for_link5_1"/>
   </joint>
+  <!-- imu_block4 -->
+  <link name="imu_block4">
+    <collision>
+      <origin xyz="0 0 0" rpy="0 0 0"/>
+      <geometry>
+        <box size="0.015 0.025 0.005"/>
+      </geometry>
+    </collision>
+    <visual>
+      <origin xyz="0 0 0" rpy="0 0 0"/>
+      <geometry>
+        <box size="0.015 0.025 0.005"/>
+      </geometry>
+      <material name="black"/>
+    </visual>
+    <xacro:default_inertial mass="1e-5"/>
+  </link>
+  <joint name="for_link5_1_to_imu_block4" type="fixed">
+    <origin xyz="0 0 ${0.005/2 + for_link5_h/2}" rpy="0 0 0"/>
+    <parent link="for_link5_1"/>
+    <child link="imu_block4"/>
+  </joint>
   <!-- link5 -->
   <link name="link5">
@@ -320,4 +408,46 @@
     <child link="for_link5_2"/>
   </joint>
+  <!-- imu_block5 -->
+  <link name="imu_block5">
+    <collision>
+      <origin xyz="0 0 0" rpy="0 0 0"/>
+      <geometry>
+        <box size="0.015 0.025 0.005"/>
+      </geometry>
+    </collision>
+    <visual>
+      <origin xyz="0 0 0" rpy="0 0 0"/>
+      <geometry>
+        <box size="0.015 0.025 0.005"/>
+      </geometry>
+      <material name="black"/>
+    </visual>
+    <xacro:default_inertial mass="1e-5"/>
+  </link>
+  <joint name="for_link5_2_to_imu_block5" type="fixed">
+    <origin xyz="0 0 ${-0.005/2 - for_link5_h/2}" rpy="0 0 0"/>
+    <parent link="for_link5_2"/>
+    <child link="imu_block5"/>
+  </joint>
+ <!-- laser4 -->
+  <link name="laser4">
+    <collision>
+      <geometry>
+        <box size="0.001 0.005 0.002"/>
+      </geometry>
+    </collision>
+    <visual>
+      <geometry>
+        <box size="0.001 0.005 0.002"/>
+      </geometry>
+      <material name="black"/>
+    </visual>
+    <xacro:default_inertial mass="1e-5"/>
+  </link>
+  <joint name="for_link5_2_to_laser4" type="fixed">
+    <origin xyz="${-link5_w/2/2 - 0.001/2} 0 0" rpy="0 3.14 0"/>
+    <parent link="for_link5_2"/>
+    <child link="laser4"/>
+  </joint>
   <!-- GRIPPER -->
   <!-- right_finger -->
@@ -457,23 +587,23 @@
     <child link="for_laser_right_2"/>
   </joint>
-  <!-- laser_right -->
-  <link name="laser_right">
-    <collision>
-      <geometry>
-        <box size="0.001 0.005 0.002"/>
-      </geometry>
-    </collision>
-    <visual>
-      <geometry>
-        <box size="0.001 0.005 0.002"/>
-      </geometry>
-      <material name="black"/>
-    </visual>
-    <xacro:default_inertial mass="1e-5"/>
-  </link>
-  <joint name="for_laser_right_2_to_laser_right" type="fixed">
+  <!-- laser3 -->
+  <link name="laser3">
+    <collision>
+      <geometry>
+        <box size="0.001 0.005 0.002"/>
+      </geometry>
+    </collision>
+    <visual>
+      <geometry>
+        <box size="0.001 0.005 0.002"/>
+      </geometry>
+      <material name="black"/>
+    </visual>
+    <xacro:default_inertial mass="1e-5"/>
+  </link>
+  <joint name="for_laser_right_2_to_laser3" type="fixed">
     <origin xyz="${-0.065/4} ${-0.001/2 - 0.002/2} 0" rpy="0 0 -1.57"/>
     <parent link="for_laser_right_2"/>
-    <child link="laser_right"/>
+    <child link="laser3"/>
   </joint>
   <!-- for_laser_left_1 -->
@@ -519,23 +649,23 @@
     <child link="for_laser_left_2"/>
   </joint>
-  <!-- laser_left -->
-  <link name="laser_left">
-    <collision>
-      <geometry>
-        <box size="0.001 0.005 0.002"/>
-      </geometry>
-    </collision>
-    <visual>
-      <geometry>
-        <box size="0.001 0.005 0.002"/>
-      </geometry>
-      <material name="black"/>
-    </visual>
-    <xacro:default_inertial mass="1e-5"/>
-  </link>
-  <joint name="for_laser_left_2_to_laser_left" type="fixed">
+  <!-- laser2 -->
+  <link name="laser2">
+    <collision>
+      <geometry>
+        <box size="0.001 0.005 0.002"/>
+      </geometry>
+    </collision>
+    <visual>
+      <geometry>
+        <box size="0.001 0.005 0.002"/>
+      </geometry>
+      <material name="black"/>
+    </visual>
+    <xacro:default_inertial mass="1e-5"/>
+  </link>
+  <joint name="for_laser_left_2_to_laser2" type="fixed">
     <origin xyz="${-0.065/4} ${0.001/2 + 0.002/2} 0" rpy="0 0 1.57"/>
     <parent link="for_laser_left_2"/>
-    <child link="laser_left"/>
+    <child link="laser2"/>
   </joint>
 </robot>
